Commit message: xacro include

File: turtlebot4_description/urdf/sensors/light_sensor.urdf.xacro (robot description, xacro)
@@ -3,6 +3,6 @@
 <xacro:macro name="light_sensor" params="name" >
   <gazebo>
-		<model name="${name}">
-			<static>true</static>
+		<!--<model name="${name}">-->
+			<!--<static>true</static>-->
 			<link name="${name}_link">
 				<visual name="visual_object">
@@ -24,6 +24,6 @@
 				<update_rate>1</update_rate>
 			</plugin>
-    </model>
-  <gazebo>
+    <!--</model>-->
+  </gazebo>
 </xacro:macro>
 </robot>

File: turtlebot4_description/urdf/standard/turtlebot4.urdf.xacro (robot description, xacro)
@@ -101,28 +101,5 @@
     <origin xyz="${oakd_pro_x_offset} ${oakd_pro_y_offset} ${oakd_pro_z_offset}"/>
   </xacro:oakd>
-  <gazebo>
-		<model name="light_sensor">
-			<static>true</static>
-      <joint name="light_joint">
-			<link name="light_sensor_link">
-				<visual name="visual_object">
-					<geometry>
-						<cylinder>
-							<radius>.1</radius>
-							<length>0.08</length>
-						</cylinder>
-						</geometry>
-						<material>
-							<diffuse>1 0 0 1</diffuse>
-						</material>
-				</visual>
-      </link>
-			<!--FIXME no absoulte path-->
-			<plugin
-				filename="/home/paolo/light_sensor_plugin/install/lib/libLightSensor.so"
-				name="custom_light_sensor::LightSensor">
-				<update_rate>1</update_rate>
-			</plugin>
-    </model>
-  </gazebo>
+  <xacro:include filename="$(find turtlebot4_description)/urdf/sensors/light_sensor.urdf.xacro" />
+  <xacro:light_sensor name="light_sensor" />
 </robot>

Commit message: fixed light sensor
fixed light sensor but the solution scales really badly

File: turtlebot4_description/urdf/sensors/light_sensor.urdf.xacro (robot description, xacro)
@@ -1,21 +1,33 @@
 <?xml version="1.0"?>
 <robot xmlns:xacro="http://ros.org/wiki/xacro">
-<xacro:macro name="light_sensor" params="name" >
+<xacro:macro name="light_sensor" params="name">
   <gazebo>
 		<!--<model name="${name}">-->
 			<!--<static>true</static>-->
 			<link name="${name}_link">
+			<pose> 0.1 0 0.35 0 0 0 </pose>
 				<visual name="visual_object">
 					<geometry>
 						<cylinder>
-							<radius>.1</radius>
-							<length>0.08</length>
+							<radius>0.01</radius>
+							<length>0.01</length>
 						</cylinder>
 						</geometry>
 						<material>
-							<diffuse>1 0 0 1</diffuse>
+							<diffuse>0 1 1 1</diffuse>
 						</material>
 				</visual>
-      </link>
+				<inertial>
+					<inertia>
+						<ixx>0</ixx>
+						<ixy>0</ixy>
+						<ixz>0</ixz>
+						<iyy>0</iyy>
+						<iyz>0</iyz>
+						<izz>0</izz>
+					</inertia>
+					<mass>0.1</mass>
+				</inertial>
+      		</link>
 			<!--FIXME no absoulte path-->
 			<plugin

File: turtlebot4_description/urdf/standard/turtlebot4.urdf.xacro (robot description, xacro)
@@ -90,5 +90,5 @@
     <origin xyz="0 0 ${tower_sensor_plate_z_offset}"/>
   </xacro:tower_sensor_plate>
-  <!-- Turtlebot4 sensor definitions -->
+  <!-- Turtlebot4 sensors definitions -->
   <xacro:rplidar name="rplidar" parent_link="shell_link" gazebo="$(arg gazebo)">
     <origin xyz="${rplidar_x_offset} ${rplidar_y_offset} ${rplidar_z_offset}"
@@ -101,5 +101,11 @@
     <origin xyz="${oakd_pro_x_offset} ${oakd_pro_y_offset} ${oakd_pro_z_offset}"/>
   </xacro:oakd>
+  <gazebo>
+    <joint name="light_joint" type="fixed">
+      <parent>base_link</parent>
+      <child>light_sensor1_link</child>
+    </joint>
+  </gazebo>
   <xacro:include filename="$(find turtlebot4_description)/urdf/sensors/light_sensor.urdf.xacro" />
-  <xacro:light_sensor name="light_sensor" />
+  <xacro:light_sensor name="light_sensor1"/>
 </robot>

Commit message: added second light sensor

File: turtlebot4_description/urdf/sensors/light_sensor.urdf.xacro (robot description, xacro)
@@ -2,9 +2,8 @@
 <robot xmlns:xacro="http://ros.org/wiki/xacro">
 <xacro:macro name="light_sensor" params="name">
-  <gazebo>
-		<!--<model name="${name}">-->
-			<!--<static>true</static>-->
+	<gazebo>
+		<model name="${name}">
+			<pose> 0.1 0 0.35 0 0 0 </pose>
 			<link name="${name}_link">
-			<pose> 0.1 0 0.35 0 0 0 </pose>
 				<visual name="visual_object">
 					<geometry>
@@ -29,13 +28,13 @@
 					<mass>0.1</mass>
 				</inertial>
-      		</link>
+	    	</link>
 			<!--FIXME no absoulte path-->
 			<plugin
 				filename="/home/paolo/light_sensor_plugin/install/lib/libLightSensor.so"
 				name="custom_light_sensor::LightSensor">
-				<update_rate>1</update_rate>
+				<update_rate>5</update_rate>
 			</plugin>
-    <!--</model>-->
-  </gazebo>
+		</model>
+	</gazebo>
 </xacro:macro>
 </robot>

File: turtlebot4_description/urdf/standard/turtlebot4.urdf.xacro (robot description, xacro)
@@ -101,11 +101,81 @@
     <origin xyz="${oakd_pro_x_offset} ${oakd_pro_y_offset} ${oakd_pro_z_offset}"/>
   </xacro:oakd>
+  <!--include light sensors-->
+  <!--<xacro:include filename="$(find turtlebot4_description)/urdf/sensors/light_sensor.urdf.xacro" />
+  <xacro:light_sensor name="light_sensor1"/>-->
+  <!--<joint name="light_joint" type="fixed">
+    <parent link="base_link"/>
+    <child link="shell_link"/>
+    <origin xyz="0 0 ${shell_z_offset + base_link_z_offset}" rpy="0 0 0"/>
+  </joint>-->
   <gazebo>
-    <joint name="light_joint" type="fixed">
-      <parent>base_link</parent>
-      <child>light_sensor1_link</child>
-    </joint>
+    <!-- light sensor 1-->
+    <model name="light_sensor1">
+	    <link name="light_link1">
+	      <pose> 0.1 0 0.35 0 0 0 </pose>
+	    	<visual name="visual_object1">
+	    		<geometry>
+	    			<cylinder>
+	    				<radius>0.01</radius>
+	    				<length>0.01</length>
+	    			</cylinder>
+	    			</geometry>
+	    			<material>
+	    				<diffuse>0 1 1 1</diffuse>
+	    			</material>
+	    	</visual>
+	    	<inertial>
+	    		<inertia>
+	    			<ixx>0</ixx>
+	    			<ixy>0</ixy>
+	    			<ixz>0</ixz>
+	    			<iyy>0</iyy>
+	    			<iyz>0</iyz>
+	    			<izz>0</izz>
+	    		</inertia>
+	    		<mass>0.1</mass>
+	    	</inertial>
+      </link>
+		  	<!--FIXME no absoulte path-->
+		  	<plugin
+		  		filename="/home/paolo/light_sensor_plugin/install/lib/libLightSensor.so"
+		  		name="custom_light_sensor::LightSensor">
+		  		<update_rate>5</update_rate>
+		  	</plugin>
+    </model>
+    <!-- light sensor 2-->
+    <model name="light_sensor2">
+	    <link name="light_link2">
+	      <pose> -0.1 0 0.35 0 0 0 </pose>
+	    	<visual name="visual_object2">
+	    		<geometry>
+	    			<cylinder>
+	    				<radius>0.01</radius>
+	    				<length>0.01</length>
+	    			</cylinder>
+	    			</geometry>
+	    			<material>
+	    				<diffuse>0 0 1 1</diffuse>
+	    			</material>
+	    	</visual>
+	    	<inertial>
+	    		<inertia>
+	    			<ixx>0</ixx>
+	    			<ixy>0</ixy>
+	    			<ixz>0</ixz>
+	    			<iyy>0</iyy>
+	    			<iyz>0</iyz>
+	    			<izz>0</izz>
+	    		</inertia>
+	    		<mass>0.1</mass>
+	    	</inertial>
+      </link>
+		  	<!--FIXME no absoulte path-->
+		  	<plugin
+		  		filename="/home/paolo/light_sensor_plugin/install/lib/libLightSensor.so"
+		  		name="custom_light_sensor::LightSensor">
+		  		<update_rate>5</update_rate>
+		  	</plugin>
+    </model>
   </gazebo>
-  <xacro:include filename="$(find turtlebot4_description)/urdf/sensors/light_sensor.urdf.xacro" />
-  <xacro:light_sensor name="light_sensor1"/>
 </robot>
