Commit message: added light

File: turtlebot4_description/urdf/standard/turtlebot4.urdf.xacro (robot description, xacro)
@@ -101,3 +101,28 @@
     <origin xyz="${oakd_pro_x_offset} ${oakd_pro_y_offset} ${oakd_pro_z_offset}"/>
   </xacro:oakd>
+  <gazebo>
+		<model name="light_sensor">
+			<static>true</static>
+      <joint name="light_joint">
+			<link name="light_sensor_link">
+				<visual name="visual_object">
+					<geometry>
+						<cylinder>
+							<radius>.1</radius>
+							<length>0.08</length>
+						</cylinder>
+						</geometry>
+						<material>
+							<diffuse>1 0 0 1</diffuse>
+						</material>
+				</visual>
+      </link>
+			<!--FIXME no absoulte path-->
+			<plugin
+				filename="/home/paolo/light_sensor_plugin/install/lib/libLightSensor.so"
+				name="custom_light_sensor::LightSensor">
+				<update_rate>1</update_rate>
+			</plugin>
+    </model>
+  </gazebo>
 </robot>

Commit message: added the deatchable_joint for the objects with namespace suppot

File: turtlebot4_description/urdf/standard/turtlebot4.urdf.xacro (robot description, xacro)
@@ -1,4 +1,6 @@
 <?xml version="1.0" ?>
 <robot name="turtlebot4" xmlns:xacro="http://ros.org/wiki/xacro">
+  <xacro:arg name="namespace" default="turtlebot4"/>
+  <xacro:property name="robot_ns" value="$(arg namespace)"/>
   <!-- Base create3 model -->
   <xacro:include filename="$(find irobot_create_description)/urdf/create3.urdf.xacro" />
@@ -90,4 +92,17 @@
     <origin xyz="0 0 ${tower_sensor_plate_z_offset}"/>
   </xacro:tower_sensor_plate>
+<!-- DetachableJoint: una istanza per ogni oggetto -->
+  <gazebo>
+    <!-- object1 detachable link-->
+    <plugin filename="gz-sim-detachable-joint-system"
+            name="gz::sim::systems::DetachableJoint">
+      <parent_link>tower_sensor_plate</parent_link>          <!-- link del robot -->
+      <child_model>object1</child_model>                     <!-- nome MODEL nel world -->
+      <child_link>link_object</child_link>       <!-- link interno dell'oggetto -->
+      <attach_topic>/${robot_ns}/object1/attach</attach_topic>
+      <detach_topic>/${robot_ns}/object1/detach</detach_topic>
+      <output_topic>/${robot_ns}/object1/state</output_topic>
+    </plugin>
+  </gazebo>
   <!-- Turtlebot4 sensor definitions -->
   <xacro:rplidar name="rplidar" parent_link="shell_link" gazebo="$(arg gazebo)">
